File: UKW TX/UKW TX.sch (KiCad schematic (older format))
At the start: 13 parts

Commit message: layout quasi fertig.
Parts:
- added C1, C3, C7, C8: 100n, Capacitors_SMD:C_0402, symbol C
- added C16, C17: 100p, Capacitors_SMD:C_0402, symbol C
- added C2, C6: 22µ, Capacitors_SMD:C_0805, symbol C
- added C4, C5, C9: 1nF, Capacitors_SMD:C_0805, symbol C
- added CON1: BARREL_JACK, symbol BARREL_JACK
- added D1: 1n4148, Diodes_SMD:Diode-MiniMELF_Standard, symbol D
- added D2: grün, LEDs:LED-0603, symbol LED
- added L1: 10µH, Resistors_SMD:R_0805, symbol INDUCTOR_SMALL
- added L2: 470nH, Resistors_SMD:R_1206, symbol INDUCTOR_SMALL
- added P1, P2: CONN_01X01, Pin_Headers:Pin_Header_Angled_1x01, symbol CONN_01X01
- added P3: CONN_01X05, Pin_Headers:Pin_Header_Angled_1x05, symbol CONN_01X05
- added R1: 100, Capacitors_SMD:C_0603, symbol R
- added R2: 220, Resistors_SMD:R_0603, symbol R
- added R5, R6: 1k, Resistors_SMD:R_0402, symbol R
- added SMA_E1: Platinenkantenbuchse, SMA_EDGE:SMA_EDGE, symbol SMA_EDGE
- added T1: TRANSFO, BA_Bauteile:AT224-1A, symbol TRANSFO
- added U1: AP1117D33, Housings_SOT-89:SOT89-3_Housing, symbol AP1117D33
- added U2: THS9001, Housings_SOT-23_SOT-143_TSOT-6:SOT-23-6, symbol THS9001
- L3, L4, L5: renamed from L?; footprint (none) -> Resistors_SMD:R_0805
- U3: renamed from U?; footprint (none) -> Alps603A:Alps_603A
- Y1: renamed from Y?; footprint (none) -> Resistors_SMD:R_1206
- gave numbers to parts that had none: 8
Connections:
- net +3V3: now also C3.1, D1.2 (A), D2.2 (A), U1.2 (VO)
- net GND: now also U3.17 (F192), C1.2, C16.2, C17.2, C2.2, C3.2, C6.2, C7.2, C8.2, CON1.1, L2.1, P3.5 (P5), R1.2, SMA_E1.0 (GND), SMA_E1.2 (GND), T1.1 (AA), U1.1 (GND/ADJ), U2.2 (GND)
- net RDS: now also P3.4 (P4)
- net SCL: now also P3.3 (P3)
- net SDA: now also P3.2 (P2)
- net Ton_L: now also CON1.2, R5.2; no longer U3.21 (Audio_L)
- net Ton_R: now also CON1.3, R6.1; no longer U3.22 (Audio_R)
- net at U3.2 (FM_Out): now also C9.2
- new net: C17.1, R5.1, U3.21 (Audio_L)
- new net: C16.1, R6.2, U3.22 (Audio_R)
- new net: C9.1, U2.1 (IF)
- new net: C8.1, U2.3 (Vs)
- new net: L2.2, U2.4 (Lcol)
- new net: C4.2, C5.2, U2.5 (IFout)
- new net: R2.2, U2.6 (BIAS)
- new net: C6.1, C7.1, L1.1, R2.1
- new net: P1.1 (P1), T1.2 (AB)
- new net: P2.1 (P1), T1.3 (SA)
- new net: C4.1, T1.4 (SB)
- new net: D2.1 (K), R1.1
- new net: C5.1, SMA_E1.1 (SIGNAL)
- new net +5V: C1.1, C2.1, D1.1 (K), L1.2, P3.1 (P1), U1.3 (VI)
- no-connect marks 1 -> 0
Other:
- note added: "3,3V werden hier selbergemacht.\nder Raspi liefert zu wenig Power."
- note added: "3,5mm Klinkenbuchse"
- note added: "50 Ohm shielded stripline"
- note added: "Es wird davon ausgegangen,\ndass die 5V-Versorgung einiger-\ngermaßen glatt ist. Trotzdem\nkommt eine Spule in die\nVersorgungsleitung."
- note added: "Raspi hier anschließen"
- note added: "kurze Leitung!"
- moved on the sheet: C10, C11, C12, C13, C14, C15, L3, L4, L5, R3, R4, U3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

Commit message: platine fertig.
Parts:
- CON1: footprint (none) -> lpis2812:LUM1503
Changed lines of the file:
@@
 F 0 "CON1" H 10050 3350 60  0000 C CNN
 F 1 "BARREL_JACK" H 10050 2900 60  0000 C CNN
-F 2 "" H 10050 3100 60  0001 C CNN
+F 2 "lpis2812:LUM1503" H 10050 3100 60  0001 C CNN
 F 3 "" H 10050 3100 60  0000 C CNN
 	1    10050 3100
